Commit message: changed original files to fitt TB

File: src/turtlebot3_manipulation_description/urdf/open_manipulator_x.urdf.xacro (robot description, xacro)
@@ -157,5 +157,5 @@
       <origin xyz="0.0817 0.021 0.0" rpy="0 0 0"/>
       <axis xyz="0 1 0"/>
-      <limit velocity="4.8" effort="1" lower="-0.010" upper="0.019" />
+      <limit velocity="4.8" effort="1" lower="-0.004" upper="0.019" />
       <dynamics damping="0.1"/>
     </joint>
@@ -192,5 +192,5 @@
       <origin xyz="0.0817 -0.021 0" rpy="0 0 0"/>
       <axis xyz="0 -1 0"/>
-      <limit velocity="4.8" effort="1" lower="-0.010" upper="0.019" />
+      <limit velocity="4.8" effort="1" lower="-0.004" upper="0.019" />
       <mimic joint="${prefix}gripper_left_joint" multiplier="1"/>
       <dynamics damping="0.1"/>

File: src/turtlebot3_manipulation_description/urdf/turtlebot3_manipulation.urdf.xacro (robot description, xacro)
@@ -24,5 +24,5 @@
     <parent link="$(arg prefix)base_link"/>
     <child link="$(arg prefix)link1"/>
-    <origin xyz="-0.092 0.0 0.091" rpy="0 0 0"/>
+    <origin xyz="0.00 0.035 0.144" rpy="0 0 -1.57"/>
   </joint>
   <xacro:open_manipulator_x prefix="$(arg prefix)" />

Commit message: Added analog and joint position

File: src/turtlebot3_manipulation_description/urdf/open_manipulator_x.urdf.xacro (robot description, xacro)
@@ -157,5 +157,5 @@
       <origin xyz="0.0817 0.021 0.0" rpy="0 0 0"/>
       <axis xyz="0 1 0"/>
-      <limit velocity="4.8" effort="1" lower="-0.004" upper="0.019" />
+      <limit velocity="4.8" effort="1" lower="-0.010" upper="0.019" />
       <dynamics damping="0.1"/>
     </joint>
@@ -192,5 +192,5 @@
       <origin xyz="0.0817 -0.021 0" rpy="0 0 0"/>
       <axis xyz="0 -1 0"/>
-      <limit velocity="4.8" effort="1" lower="-0.004" upper="0.019" />
+      <limit velocity="4.8" effort="1" lower="-0.010" upper="0.019" />
       <mimic joint="${prefix}gripper_left_joint" multiplier="1"/>
       <dynamics damping="0.1"/>

File: src/turtlebot3_manipulation_description/urdf/turtlebot3_manipulation.urdf.xacro (robot description, xacro)
@@ -24,5 +24,5 @@
     <parent link="$(arg prefix)base_link"/>
     <child link="$(arg prefix)link1"/>
-    <origin xyz="0.00 0.035 0.144" rpy="0 0 -1.57"/>
+    <origin xyz="-0.092 0.0 0.091" rpy="0 0 0"/>
   </joint>
   <xacro:open_manipulator_x prefix="$(arg prefix)" />
